Commit message: pi_camera

File: src/robot_description/urdf/robot.urdf.xacro (robot description, xacro)
@@ -17,4 +17,16 @@
         <child link = "base_link"/>
         <origin rpy="0 0 0" xyz=" 0 0 0"/>
+    </joint>
+    <link name="pi_camera">
+        <visual>
+            <geometry>
+                <mesh filename="package://robot_description/meshes/pi_camera.STL" scale="0.01 0.01 0.01"/>
+            </geometry>
+        </visual>
+    </link>
+    <joint name="pi_camera_joint" type="fixed">
+        <parent link="base_link"/>
+        <child link="pi_camera"/>
+        <origin rpy="0 -0.5 1.57 " xyz=" 0 0.45 0.2 "/>
     </joint>
     <link name="base_plate">

Commit message: added changes for gazebo simulations

File: src/robot_description/urdf/robot.urdf.xacro (robot description, xacro)
@@ -4,6 +4,15 @@
     <xacro:property name="effort" value="30.0"/>
     <xacro:property name="velocity" value="10.0"/>
+    <xacro:macro name="default_inertia" params="mass">
+        <inertial>
+            <mass value="${mass}"/>
+            <inertia ixx="1.0" ixy="0.0" ixz="0.0"
+                     iyy="1.0" iyz="0.0"
+                     izz="1.0" />
+        </inertial>
+    </xacro:macro>
     <link name="world"/>
     <link name="base_link">
+        <xacro:default_inertia mass="1.0"/>
         <visual>
             <origin rpy="0 0 0" xyz="-0.5 -0.5 0"/>
@@ -12,4 +21,10 @@
             </geometry>
         </visual>
+        <collision>
+            <origin rpy="0 0 0" xyz="-0.5 -0.5 0"/>
+            <geometry>
+                <mesh filename="package://robot_description/meshes/basement.STL" scale="0.01 0.01 0.01"/>
+            </geometry>
+        </collision>
     </link>
     <joint name="virtual_joint" type="fixed">
@@ -19,9 +34,17 @@
     </joint>
     <link name="pi_camera">
+        <xacro:default_inertia mass="0.1"/>
         <visual>
+            <origin rpy="-1.57 0 -1.57" xyz="-0.1 0.125 0.14"/>
             <geometry>
                 <mesh filename="package://robot_description/meshes/pi_camera.STL" scale="0.01 0.01 0.01"/>
             </geometry>
         </visual>
+        <collision>
+            <origin rpy="-1.57 0 -1.57" xyz="-0.1 0.125 0.14"/>
+            <geometry>
+                <mesh filename="package://robot_description/meshes/pi_camera.STL" scale="0.01 0.01 0.01"/>
+            </geometry>
+        </collision>
     </link>
     <joint name="pi_camera_joint" type="fixed">
@@ -31,4 +54,5 @@
     </joint>
     <link name="base_plate">
+        <xacro:default_inertia mass="0.1"/>
         <visual>
             <origin rpy=" 0 0 0" xyz="-0.39 -0.39 -0.56"/>
@@ -37,4 +61,10 @@
             </geometry>
         </visual>
+        <collision>
+            <origin rpy=" 0 0 0" xyz="-0.39 -0.39 -0.56"/>
+            <geometry>
+                <mesh filename="package://robot_description/meshes/base_plate.STL" scale="0.01 0.01 0.01"/>
+            </geometry>
+        </collision>
     </link>
     <joint name="joint_1" type="revolute">
@@ -46,4 +76,5 @@
     </joint>
     <link name="forward_drive_arm">
+        <xacro:default_inertia mass="0.1"/>
         <visual>
             <origin rpy=" 0 -${PI/2} ${PI/2}" xyz="0.19 0.06 -0.08"/>
@@ -52,4 +83,10 @@
             </geometry>
         </visual>
+        <collision>
+            <origin rpy=" 0 -${PI/2} ${PI/2}" xyz="0.19 0.06 -0.08"/>
+            <geometry>
+                <mesh filename="package://robot_description/meshes/forward_drive_arm.STL" scale="0.01 0.01 0.01"/>
+            </geometry>
+        </collision>
     </link>
     <joint name="joint_2" type="revolute">
@@ -61,4 +98,5 @@
     </joint>
     <link name="horizontal_arm">
+        <xacro:default_inertia mass="0.1"/>
         <visual>
             <origin rpy=" ${PI/2} 0 ${PI/2}" xyz="-0.03 -0.4 -0.06"/>
@@ -67,4 +105,10 @@
             </geometry>
         </visual>
+        <collision>
+            <origin rpy=" ${PI/2} 0 ${PI/2}" xyz="-0.03 -0.4 -0.06"/>
+            <geometry>
+                <mesh filename="package://robot_description/meshes/horizontal_arm.STL" scale="0.01 0.01 0.01"/>
+            </geometry>
+        </collision>
     </link>
     <joint name="joint_3" type="revolute">
@@ -76,4 +120,5 @@
     </joint>
     <link name="claw_support">
+        <xacro:default_inertia mass="0.05"/>
         <visual>
             <origin rpy=" 0 0 ${PI/2}" xyz="0 -0.05 -0.15"/>
@@ -82,4 +127,10 @@
             </geometry>
         </visual>
+        <collision>
+            <origin rpy=" 0 0 ${PI/2}" xyz="0 -0.05 -0.15"/>
+            <geometry>
+                <mesh filename="package://robot_description/meshes/claw_support.STL" scale="0.01 0.01 0.01"/>
+            </geometry>
+        </collision>
     </link>
     <joint name="horizontal_arm_to_claw_support" type="fixed">
@@ -89,4 +140,5 @@
     </joint>
     <link name="gripper_right">
+        <xacro:default_inertia mass="0.01"/>
         <visual>
             <origin rpy=" 0 0 -${PI/2}" xyz="-0.1 0.5 -0.1"/>
@@ -95,6 +147,13 @@
             </geometry>
         </visual>
+        <collision>
+            <origin rpy=" 0 0 -${PI/2}" xyz="-0.1 0.5 -0.1"/>
+            <geometry>
+                <mesh filename="package://robot_description/meshes/right_finger.STL" scale="0.01 0.01 0.01"/>
+            </geometry>
+        </collision>
     </link>
     <link name="gripper_left">
+        <xacro:default_inertia mass="0.01"/>
         <visual>
             <origin rpy=" 0 0 -${PI/2}" xyz="-0.04 0.5 -0.1"/>
@@ -103,4 +162,10 @@
             </geometry>
         </visual>
+        <collision>
+            <origin rpy=" 0 0 -${PI/2}" xyz="-0.04 0.5 -0.1"/>
+            <geometry>
+                <mesh filename="package://robot_description/meshes/left_finger.STL" scale="0.01 0.01 0.01"/>
+            </geometry>
+        </collision>
     </link>
     <joint name="joint_4" type="revolute">
